Commit message: feat: adjust_tourobo-robot

File: xacro/omni_robot.xacro (robot description, xacro)
@@ -8,9 +8,9 @@
 	<joint name="base_joint" type="fixed">
 		<parent link="base_footprint"/>
-		<child link="base_link"/>
+		<child link="base_frame"/>
 	</joint>
-	<link name="base_link"/>
+	<link name="base_frame"/>
 	<joint name="body_joint" type="fixed">
-		<parent link="base_link"/>
+		<parent link="base_frame"/>
 		<child link="body_link"/>
 		<origin xyz="0 0 0.15" rpy="0 0 0"/>
@@ -34,5 +34,5 @@
 	</link>
 	<xacro:imu_macro prefix="imu" parent="body_link" xyz="0 0 0" rpy="0 0 0"/>
-	<xacro:lidar_macro prefix="laser" parent="body_link" xyz="0 0.2 -0.10" rpy="0 0 0"/>
+	<xacro:lidar_macro prefix="laser" parent="body_link" xyz="0 0.2 -0.10" rpy="3.14159265 0 1.570796"/>
 	<xacro:wheel_macro prefix="fr_wheel" parent="body_link" xyz="0.2 0.2 -0.06"/>
 	<xacro:wheel_macro prefix="fl_wheel" parent="body_link" xyz="-0.2 0.2 -0.06"/>

File: xacro/sensor_macro.xacro (robot description, xacro)
@@ -35,5 +35,5 @@
 			<child link="${prefix}_link"/>
 		</joint>
-		<link name="${prefix}_link">
+        <link name="${prefix}_link">
 			<visual>
 				<geometry>
@@ -43,5 +43,5 @@
 		</link>
 		<gazebo reference="${prefix}_link">
-			<sensor name="${prefix}_link" type="ray">
+            <sensor name="${prefix}_link" type="ray">
 				<topic>scan</topic>
 				<ignition_frame_id>${prefix}_link</ignition_frame_id>
@@ -75,5 +75,5 @@
 					</ros>
 					<output_type>sensor_msgs/LaserScan</output_type>
-					<frame_name>${prefix}_link</frame_name>
+                    <frame_name>laser</frame_name>
 				</plugin>
 			</sensor>
